File: schematic/schematic.kicad_sch (KiCad schematic)
At the start: 15 parts, among them SW1 RED_BUTTON, SW2 BLUE_BUTTON, SW3 YELLOW_BUTTON, SW4 GREEN_BUTTON, U1 74LS48, U2 FND500

Commit message: updated schematic
Parts:
- added R5, R6: 1 kΩ, symbol Device:R
Connections:
- net at A1.6 (GND), U1.8 (GND), U2.5 (DP): now also R5.2, R6.2; no longer U2.3 (CC), U2.8 (CC)
- new net: R6.1, U2.8 (CC)
- new net: R5.1, U2.3 (CC)
Changed lines of the file:
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@@
   (junction (at 83.82 146.05) (diameter 0) (color 0 0 0 0)
   )
-  (junction (at 242.57 130.81) (diameter 0) (color 0 0 0 0)
+  (junction (at 260.35 130.81) (diameter 0) (color 0 0 0 0)
+  )
+  (wire (pts (xy 260.35 128.27) (xy 246.38 128.27))
+    (stroke (width 0) (type default))
   )
   (wire (pts (xy 105.41 67.31) (xy 130.81 67.31))
@@
     (stroke (width 0) (type default))
   )
+  (wire (pts (xy 260.35 130.81) (xy 256.54 130.81))
+    (stroke (width 0) (type default))
+  )
   (wire (pts (xy 105.41 44.45) (xy 142.24 44.45))
     (stroke (width 0) (type default))
@@
     (stroke (width 0) (type default))
   )
-  (wire (pts (xy 236.22 130.81) (xy 242.57 130.81))
-    (stroke (width 0) (type default))
-  )
   (wire (pts (xy 104.14 123.19) (xy 104.14 146.05))
     (stroke (width 0) (type default))
@@
     (stroke (width 0) (type default))
   )
+  (wire (pts (xy 238.76 128.27) (xy 236.22 128.27))
+    (stroke (width 0) (type default))
+  )
   (wire (pts (xy 180.34 97.79) (xy 198.12 97.79))
     (stroke (width 0) (type default))
@@
     (stroke (width 0) (type default))
   )
-  (wire (pts (xy 236.22 128.27) (xy 242.57 128.27))
-    (stroke (width 0) (type default))
-  )
   (wire (pts (xy 210.82 113.03) (xy 220.98 113.03))
     (stroke (width 0) (type default))
@@
     (stroke (width 0) (type default))
   )
+  (wire (pts (xy 236.22 130.81) (xy 248.92 130.81))
+    (stroke (width 0) (type default))
+  )
   (wire (pts (xy 140.97 87.63) (xy 140.97 113.03))
     (stroke (width 0) (type default))
   )
-  (wire (pts (xy 242.57 130.81) (xy 242.57 140.97))
+  (wire (pts (xy 260.35 130.81) (xy 260.35 140.97))
     (stroke (width 0) (type default))
   )
@@
     (stroke (width 0) (type default))
   )
-  (wire (pts (xy 242.57 128.27) (xy 242.57 130.81))
+  (wire (pts (xy 260.35 128.27) (xy 260.35 130.81))
     (stroke (width 0) (type default))
   )
@@
     (stroke (width 0) (type default))
   )
-  (wire (pts (xy 242.57 140.97) (xy 219.71 140.97))
+  (wire (pts (xy 260.35 140.97) (xy 219.71 140.97))
     (stroke (width 0) (type default))
   )
@@
     )
   )
+  (symbol (lib_id "Device:R") (at 252.73 130.81 90) (unit 1)
+    (in_bom yes) (on_board yes) (dnp no)
+    (property "Reference" "R6" (at 252.73 133.35 90)
+      (effects (font (size 1.27 1.27)))
+    )
+    (property "Value" "1 kΩ" (at 252.73 135.89 90)
+      (effects (font (size 1.27 1.27)))
+    )
+    (property "Footprint" "" (at 252.73 132.588 90)
+      (effects (font (size 1.27 1.27)) hide)
+    )
+    (property "Datasheet" "~" (at 252.73 130.81 0)
+      (effects (font (size 1.27 1.27)) hide)
+    )
+    (pin "1")
+    (pin "2")
+    (instances
+      (project "schematic"
+        (path "/ac039a42-e01f-45ad-a0b0-501ff75ecbb5"
+          (reference "R6") (unit 1)
+        )
+      )
+    )
+  )
   (symbol (lib_id "Switch:SW_Push") (at 100.33 44.45 0) (unit 1)
     (in_bom yes) (on_board yes) (dnp no)
@@
         )
       )
+    )
+  )
+  (symbol (lib_id "Device:R") (at 242.57 128.27 90) (unit 1)
+    (in_bom yes) (on_board yes) (dnp no)
+    (property "Reference" "R5" (at 242.57 123.19 90)
+      (effects (font (size 1.27 1.27)))
+    )
+    (property "Value" "1 kΩ" (at 242.57 125.73 90)
+      (effects (font (size 1.27 1.27)))
+    )
+    (property "Footprint" "" (at 242.57 130.048 90)
+      (effects (font (size 1.27 1.27)) hide)
+    )
+    (property "Datasheet" "~" (at 242.57 128.27 0)
+      (effects (font (size 1.27 1.27)) hide)
+    )
+    (pin "1")
+    (pin "2")
+    (instances
+      (project "schematic"
+        (path "/ac039a42-e01f-45ad-a0b0-501ff75ecbb5"
+          (reference "R5") (unit 1)
+        )
+      )

Commit message: added led names
Parts:
- D1: value LED -> RED_LED
- D2: value LED -> BLUE_LED
- D3: value LED -> YELLOW_LED
- D4: value LED -> GREEN_LED
Changed lines of the file:
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@@
       (effects (font (size 1.27 1.27)))
     )
-    (property "Value" "LED" (at 78.74 90.17 90)
+    (property "Value" "BLUE_LED" (at 78.74 88.9 90)
       (effects (font (size 1.27 1.27)))
     )
@@
       (effects (font (size 1.27 1.27)))
     )
-    (property "Value" "LED" (at 99.06 100.33 90)
+    (property "Value" "GREEN_LED" (at 102.87 99.06 90)
       (effects (font (size 1.27 1.27)))
     )
@@
       (effects (font (size 1.27 1.27)))
     )
-    (property "Value" "LED" (at 68.58 82.55 90)
+    (property "Value" "RED_LED" (at 67.31 82.55 90)
       (effects (font (size 1.27 1.27)))
     )
@@
       (effects (font (size 1.27 1.27)))
     )
-    (property "Value" "LED" (at 88.9 95.25 90)
-      (effects (font (size 1.27 1.27)))
-    )
+    (property "Value" "YELLOW_LED" (at 92.71 93.98 90)
+      (effects (font (size 1.27 1.27)))
+    )
